Commit message: added gazebo launch files

File: gp8_description/urdf/control/gp8_ro2_control.urdf.xacro (robot description, xacro)
@@ -1,5 +1,5 @@
 <?xml version="1.0" ?>
 <robot xmlns:xacro="http://wiki.ros.org/xacro">
-    <xacro:macro name="gp8_ros2_control" params="prefix use_gazebo">
+    <xacro:macro name="motoman_gp8_ros2_control" params="prefix use_gazebo">
         <ros2_control name="RobotSystem" type="system">
             <hardware>

File: gp8_description/urdf/robots/gp8.xacro (robot description, xacro)
@@ -8,5 +8,5 @@
         use_gazebo="$(arg use_gazebo)"/>
     <xacro:include filename="$(find gp8_description)/urdf/control/gp8_ros2_control.urdf.xacro" />
-    <xacro:mycobot_ros2_control
+    <xacro:motoman_gp8_ros2_control
         prefix="$(arg prefix)"
         use_gazebo="$(arg use_gazebo)"/>
