Commit message: coordinated gripper joint

File: gp8_description/urdf/control/gp8_ros2_control.urdf.xacro (robot description, xacro)
@@ -50,4 +50,21 @@
                 <state_interface name="position"/>
             </joint>
+            <joint name="${prefix}gripper_controller">
+                <command_interface name="position">
+                    <param name="min">0</param>
+                    <param name="max">0.032</param>
+                </command_interface>
+                <state_interface name="position"/>
+            </joint>
+            <joint name="${prefix}gripper_base_to_${prefix}gripper_right">
+                <param name="mimic">gripper_controller</param>
+                <param name="multiplier">1.0</param>
+                <state_interface name="position"/>
+            </joint>
+            <joint name="${prefix}gripper_base_to_${prefix}gripper_left">
+                <param name="mimic">gripper_controller</param>
+                <param name="multiplier">1.0</param>
+                <state_interface name="position"/>
+            </joint>
         </ros2_control>
     </xacro:macro>

File: gp8_description/urdf/mech/pneumatic_gripper.urdf.xacro (robot description, xacro)
@@ -160,4 +160,8 @@
       <axis
         xyz="1 0 0" />
+      <mimic
+        joint="${prefix}gripper_base_to_${prefix}gripper_right"
+        multiplier="1.0"
+        offset="0.0" />
       <limit
         lower="0"

Commit message: gazebo gripper

File: gp8_description/urdf/control/gp8_ros2_control.urdf.xacro (robot description, xacro)
@@ -50,5 +50,5 @@
                 <state_interface name="position"/>
             </joint>
-            <joint name="${prefix}gripper_controller">
+            <joint name="${prefix}gripper_base_to_${prefix}gripper_right">
                 <command_interface name="position">
                     <param name="min">0</param>
@@ -56,14 +56,9 @@
                 </command_interface>
                 <state_interface name="position"/>
+                <state_interface name="velocity"/>
             </joint>
-            <joint name="${prefix}gripper_base_to_${prefix}gripper_right">
-                <param name="mimic">gripper_controller</param>
-                <param name="multiplier">1.0</param>
+            <joint name="${prefix}gripper_base_to_${prefix}gripper_left" mimic="true" mimic_joint="${prefix}gripper_base_to_${prefix}gripper_right" multiplier="1.0">
                 <state_interface name="position"/>
-            </joint>
-            <joint name="${prefix}gripper_base_to_${prefix}gripper_left">
-                <param name="mimic">gripper_controller</param>
-                <param name="multiplier">1.0</param>
-                <state_interface name="position"/>
+                <state_interface name="velocity"/>
             </joint>
         </ros2_control>

File: gp8_description/urdf/mech/pneumatic_gripper.urdf.xacro (robot description, xacro)
@@ -102,6 +102,6 @@
         lower="0"
         upper="0.032"
-        effort="5"
-        velocity="0.2" />
+        effort="100.0"
+        velocity="1.0" />
       <dynamics
         damping="0"
@@ -167,6 +167,6 @@
         lower="0"
         upper="0.032"
-        effort="5"
-        velocity="0.2" />
+        effort="100.0"
+        velocity="1.0" />
       <dynamics
         damping="0"

File: gp8_description/urdf/robots/gp8.xacro (robot description, xacro)
@@ -26,5 +26,5 @@
             <xacro:include filename="$(find gp8_description)/urdf/mech/pneumatic_gripper.urdf.xacro"/>
             <xacro:pneumatic_gripper
-                parent="$(arg tool_link)"
+                parent="$(arg prefix)$(arg tool_link)"
                 prefix="$(arg prefix)">
                 <origin xyz="-0.005 0 0.04" rpy="${radians(90)} 0 ${radians(90)}"/>
