Commit message: added temporary inertial data

File: gp8_description/urdf/mech/gp8_macro.xacro (robot description, xacro)
@@ -1,4 +1,4 @@
 <?xml version="1.0" ?>
-<robot xmlns:xacro="http://ros.org/wiki/xacro">
+<robot xmlns:xacro="http://wiki.ros.org/xacro">
   <xacro:macro name="motoman_gp8" params="prefix">
     <xacro:include filename="$(find gp8_description)/urdf/resources/common_materials.xacro"/>
@@ -16,4 +16,9 @@
         </geometry>
       </collision>
+      <inertial>
+        <origin xyz="0 0 0.15" rpy="0 0 0"/>
+        <mass value="12.0"/>
+        <inertia ixx="0.157" ixy="0.0" ixz="0.0" iyy="0.157" iyz="0.0" izz="0.135"/>
+      </inertial>
     </link>
     <link name="${prefix}link_1_s">
@@ -29,4 +34,9 @@
         </geometry>
       </collision>
+      <inertial>
+        <origin xyz="0.02 0 0.15" rpy="0 0 0"/>
+        <mass value="8.0"/>
+        <inertia ixx="0.088" ixy="0.0" ixz="0.0" iyy="0.088" iyz="0.0" izz="0.057"/>
+      </inertial>
     </link>
     <link name="${prefix}link_2_l">
@@ -42,4 +52,9 @@
         </geometry>
       </collision>
+      <inertial>
+        <origin xyz="0 0 0.17" rpy="0 0 0"/>
+        <mass value="6.0"/>
+        <inertia ixx="0.076" ixy="0.0" ixz="0.0" iyy="0.076" iyz="0.0" izz="0.030"/>
+      </inertial>
     </link>
     <link name="${prefix}link_3_u">
@@ -55,4 +70,9 @@
         </geometry>
       </collision>
+      <inertial>
+        <origin xyz="0.17 0 0.02" rpy="0 0 0"/>
+        <mass value="4.0"/>
+        <inertia ixx="0.047" ixy="0.0" ixz="0.0" iyy="0.047" iyz="0.0" izz="0.012"/>
+      </inertial>
     </link>
     <link name="${prefix}link_4_r">
@@ -68,4 +88,9 @@
         </geometry>
       </collision>
+      <inertial>
+        <origin xyz="0 0 0" rpy="0 0 0"/>
+        <mass value="1.0"/>
+        <inertia ixx="0.006" ixy="0.0" ixz="0.0" iyy="0.006" iyz="0.0" izz="0.001"/>
+      </inertial>
     </link>
     <link name="${prefix}link_5_b">
@@ -81,4 +106,9 @@
         </geometry>
       </collision>
+      <inertial>
+        <origin xyz="0 0 0" rpy="0 0 0"/>
+        <mass value="0.5"/>
+        <inertia ixx="0.0007" ixy="0.0" ixz="0.0" iyy="0.0007" iyz="0.0" izz="0.0006"/>
+      </inertial>
     </link>
     <link name="${prefix}link_6_t">
@@ -94,4 +124,9 @@
         </geometry>
       </collision>
+      <inertial>
+        <origin xyz="0.02 0 0" rpy="0 0 0"/>
+        <mass value="0.5"/>
+        <inertia ixx="0.0004" ixy="0.0" ixz="0.0" iyy="0.0004" iyz="0.0" izz="0.0006"/>
+      </inertial>
     </link>
     <!-- end of link list -->

File: gp8_description/urdf/robots/gp8.xacro (robot description, xacro)
@@ -11,6 +11,14 @@
     <xacro:arg name="use_gazebo" default="false" />
     <xacro:arg name="use_gripper" default="false" />
+    <xacro:if value="$(arg add_world)">
+      <link name="world"/>
+      <joint name="$(arg prefix)virtual_joint" type="fixed">
+          <parent link="world"/>
+          <child link="$(arg prefix)$(arg base_link)"/>
+          <origin xyz="0 0 0" rpy="0 0 0"/>
+      </joint>
+    </xacro:if>
     <xacro:include filename="$(find gp8_description)/urdf/mech/gp8_macro.xacro" />
-    <xacro:motoman_gp8 prefix=""/>
+    <xacro:motoman_gp8 prefix="$(arg prefix)"/>
     <xacro:include filename="$(find gp8_description)/urdf/control/gazebo_sim_ros2_control.urdf.xacro" />
     <xacro:load_gazebo_sim_ros2_control_plugin

Commit message: fixed gazebo simulation

File: gp8_description/urdf/mech/gp8_macro.xacro (robot description, xacro)
@@ -1,4 +1,6 @@
 <?xml version="1.0" ?>
 <robot xmlns:xacro="http://wiki.ros.org/xacro">
+  <xacro:property name="joint_damping" value="0.0"/>
+  <xacro:property name="joint_friction" value="0.0"/>
   <xacro:macro name="motoman_gp8" params="prefix">
     <xacro:include filename="$(find gp8_description)/urdf/resources/common_materials.xacro"/>
@@ -7,11 +9,11 @@
       <visual>
         <geometry>
-          <mesh filename="package://gp8_description/meshes/gp8/visual/gp8_base_link.stl"/>
-        </geometry>
-        <xacro:material_yaskawa_blue/>
-      </visual>
-      <collision>
-        <geometry>
-          <mesh filename="package://gp8_description/meshes/gp8/collision/gp8_base_link.stl"/>
+          <mesh filename="file://$(find gp8_description)/meshes/gp8/visual/gp8_base_link.stl"/>
+        </geometry>
+        <xacro:material_yaskawa_blue/>
+      </visual>
+      <collision>
+        <geometry>
+          <mesh filename="file://$(find gp8_description)/meshes/gp8/collision/gp8_base_link.stl"/>
         </geometry>
       </collision>
@@ -25,11 +27,11 @@
       <visual>
         <geometry>
-          <mesh filename="package://gp8_description/meshes/gp8/visual/gp8_link_1_s.stl"/>
-        </geometry>
-        <xacro:material_yaskawa_blue/>
-      </visual>
-      <collision>
-        <geometry>
-          <mesh filename="package://gp8_description/meshes/gp8/collision/gp8_link_1_s.stl"/>
+          <mesh filename="file://$(find gp8_description)/meshes/gp8/visual/gp8_link_1_s.stl"/>
+        </geometry>
+        <xacro:material_yaskawa_blue/>
+      </visual>
+      <collision>
+        <geometry>
+          <mesh filename="file://$(find gp8_description)/meshes/gp8/collision/gp8_link_1_s.stl"/>
         </geometry>
       </collision>
@@ -43,11 +45,11 @@
       <visual>
         <geometry>
-          <mesh filename="package://gp8_description/meshes/gp8/visual/gp8_link_2_l.stl"/>
-        </geometry>
-        <xacro:material_yaskawa_blue/>
-      </visual>
-      <collision>
-        <geometry>
-          <mesh filename="package://gp8_description/meshes/gp8/collision/gp8_link_2_l.stl"/>
+          <mesh filename="file://$(find gp8_description)/meshes/gp8/visual/gp8_link_2_l.stl"/>
+        </geometry>
+        <xacro:material_yaskawa_blue/>
+      </visual>
+      <collision>
+        <geometry>
+          <mesh filename="file://$(find gp8_description)/meshes/gp8/collision/gp8_link_2_l.stl"/>
         </geometry>
       </collision>
@@ -61,11 +63,11 @@
       <visual>
         <geometry>
-          <mesh filename="package://gp8_description/meshes/gp8/visual/gp8_link_3_u.stl"/>
-        </geometry>
-        <xacro:material_yaskawa_blue/>
-      </visual>
-      <collision>
-        <geometry>
-          <mesh filename="package://gp8_description/meshes/gp8/collision/gp8_link_3_u.stl"/>
+          <mesh filename="file://$(find gp8_description)/meshes/gp8/visual/gp8_link_3_u.stl"/>
+        </geometry>
+        <xacro:material_yaskawa_blue/>
+      </visual>
+      <collision>
+        <geometry>
+          <mesh filename="file://$(find gp8_description)/meshes/gp8/collision/gp8_link_3_u.stl"/>
         </geometry>
       </collision>
@@ -79,11 +81,11 @@
       <visual>
         <geometry>
-          <mesh filename="package://gp8_description/meshes/gp8/visual/gp8_link_4_r.stl"/>
-        </geometry>
-        <xacro:material_yaskawa_blue/>
-      </visual>
-      <collision>
-        <geometry>
-          <mesh filename="package://gp8_description/meshes/gp8/collision/gp8_link_4_r.stl"/>
+          <mesh filename="file://$(find gp8_description)/meshes/gp8/visual/gp8_link_4_r.stl"/>
+        </geometry>
+        <xacro:material_yaskawa_blue/>
+      </visual>
+      <collision>
+        <geometry>
+          <mesh filename="file://$(find gp8_description)/meshes/gp8/collision/gp8_link_4_r.stl"/>
         </geometry>
       </collision>
@@ -97,11 +99,11 @@
       <visual>
         <geometry>
-          <mesh filename="package://gp8_description/meshes/gp8/visual/gp8_link_5_b.stl"/>
-        </geometry>
-        <xacro:material_yaskawa_blue/>
-      </visual>
-      <collision>
-        <geometry>
-          <mesh filename="package://gp8_description/meshes/gp8/collision/gp8_link_5_b.stl"/>
+          <mesh filename="file://$(find gp8_description)/meshes/gp8/visual/gp8_link_5_b.stl"/>
+        </geometry>
+        <xacro:material_yaskawa_blue/>
+      </visual>
+      <collision>
+        <geometry>
+          <mesh filename="file://$(find gp8_description)/meshes/gp8/collision/gp8_link_5_b.stl"/>
         </geometry>
       </collision>
@@ -115,11 +117,11 @@
       <visual>
         <geometry>
-          <mesh filename="package://gp8_description/meshes/gp8/visual/gp8_link_6_t.stl"/>
-        </geometry>
-        <xacro:material_yaskawa_blue/>
-      </visual>
-      <collision>
-        <geometry>
-          <mesh filename="package://gp8_description/meshes/gp8/collision/gp8_link_6_t.stl"/>
+          <mesh filename="file://$(find gp8_description)/meshes/gp8/visual/gp8_link_6_t.stl"/>
+        </geometry>
+        <xacro:material_yaskawa_blue/>
+      </visual>
+      <collision>
+        <geometry>
+          <mesh filename="file://$(find gp8_description)/meshes/gp8/collision/gp8_link_6_t.stl"/>
         </geometry>
       </collision>
@@ -138,4 +140,5 @@
       <axis xyz="0 0 1" />
       <limit lower="${radians(-170)}" upper="${radians(170)}" effort="150.92" velocity="${radians(455)}"/>
+      <dynamics damping="${joint_damping}" friction="${joint_friction}"/>
     </joint>
     <joint name="${prefix}joint_2_l" type="revolute">
@@ -145,4 +148,5 @@
       <axis xyz="0 1 0" />
       <limit lower="${radians(-65)}" upper="${radians(145)}" effort="176.4" velocity="${radians(385)}"/>
+      <dynamics damping="${joint_damping}" friction="${joint_friction}"/>
     </joint>
     <joint name="${prefix}joint_3_u" type="revolute">
@@ -152,4 +156,5 @@
       <axis xyz="0 -1 0" />
       <limit lower="${radians(-70)}" upper="${radians(190)}" effort="107.56" velocity="${radians(520)}"/>
+      <dynamics damping="${joint_damping}" friction="${joint_friction}"/>
     </joint>
     <joint name="${prefix}joint_4_r" type="revolute">
@@ -159,4 +164,5 @@
       <axis xyz="-1 0 0" />
       <limit lower="${radians(-190)}" upper="${radians(190)}" effort="55.86" velocity="${radians(550)}"/>
+      <dynamics damping="${joint_damping}" friction="${joint_friction}"/>
     </joint>
     <joint name="${prefix}joint_5_b" type="revolute">
@@ -166,4 +172,5 @@
       <axis xyz="0 -1 0" />
       <limit lower="${radians(-135)}" upper="${radians(135)}" effort="32.68" velocity="${radians(550)}"/>
+      <dynamics damping="${joint_damping}" friction="${joint_friction}"/>
     </joint>
     <joint name="${prefix}joint_6_t" type="revolute">
@@ -173,4 +180,5 @@
       <axis xyz="-1 0 0" />
       <limit lower="${radians(-360)}" upper="${radians(360)}" effort="22.54" velocity="${radians(1000)}"/>
+      <dynamics damping="${joint_damping}" friction="${joint_friction}"/>
     </joint>
     <!-- end of joint list -->
