Commit message: moveit

File: gp8_moveit_config/config/gp8/gp8_macro.srdf.xacro (robot description, xacro)
@@ -2,5 +2,5 @@
 <robot xmlns:xacro="http://wiki.ros.org/xacro">
     <xacro:macro name="gp8_srdf" params="prefix" >
-        <group name="gp8_arm">
+        <group name="arm">
             <joint name="$(arg prefix)virtual_joint"/>
             <joint name="$(arg prefix)joint_1_s"/>
@@ -11,5 +11,13 @@
             <joint name="$(arg prefix)joint_6_t"/>
         </group>
-        <group_state name="home" group="gp8_arm">
+        <group name="gripper">
+            <joint name="${prefix}gripper_base_to_${prefix}gripper_right"/>
+        </group>
+        <group name="arm_with_gripper">
+            <group name="arm" />
+            <group name="gripper" />
+        </group>
+        <end_effector name="gripper" parent_link="tool0" group="gripper"/>
+        <group_state name="home" group="arm">
             <joint name="$(arg prefix)joint_1_s" value="0"/>
             <joint name="$(arg prefix)joint_2_l" value="0"/>
@@ -19,4 +27,10 @@
             <joint name="$(arg prefix)joint_6_t" value="0"/>
         </group_state>
+        <group_state name="open" group="gripper">
+            <joint name="${prefix}gripper_base_to_${prefix}gripper_right" value="0.0"/>
+        </group_state>
+        <group_state name="closed" group="gripper">
+            <joint name="${prefix}gripper_base_to_${prefix}gripper_right" value="0.032"/>
+        </group_state>
         <disable_collisions link1="${prefix}base_link" link2="${prefix}link_1_s" reason="Adjacent"/>
         <disable_collisions link1="${prefix}link_1_s" link2="${prefix}link_2_l" reason="Adjacent"/>
@@ -25,4 +39,12 @@
         <disable_collisions link1="${prefix}link_4_r" link2="${prefix}link_5_b" reason="Adjacent"/>
         <disable_collisions link1="${prefix}link_5_b" link2="${prefix}link_6_t" reason="Adjacent"/>
+        <disable_collisions link1="${prefix}link_6_t" link2="${prefix}gripper_base" reason="Never"/>
+        <disable_collisions link1="${prefix}link_6_t" link2="${prefix}gripper_right" reason="Never"/>
+        <disable_collisions link1="${prefix}link_6_t" link2="${prefix}gripper_left" reason="Never"/>
+        <disable_collisions link1="${prefix}tool0" link2="${prefix}gripper_base" reason="Never"/>
+        <disable_collisions link1="${prefix}tool0" link2="${prefix}gripper_right" reason="Never"/>
+        <disable_collisions link1="${prefix}tool0" link2="${prefix}gripper_left" reason="Never"/>
+        <disable_collisions link1="${prefix}gripper_base" link2="${prefix}gripper_right" reason="Adjacent"/>
+        <disable_collisions link1="${prefix}gripper_base" link2="${prefix}gripper_left" reason="Adjacent"/>
     </xacro:macro>
 </robot>

Commit message: moveit alias

File: gp8_moveit_config/config/gp8/gp8_macro.srdf.xacro (robot description, xacro)
@@ -31,5 +31,5 @@
         </group_state>
         <group_state name="closed" group="gripper">
-            <joint name="${prefix}gripper_base_to_${prefix}gripper_right" value="0.032"/>
+            <joint name="${prefix}gripper_base_to_${prefix}gripper_right" value="0.031"/>
         </group_state>
         <disable_collisions link1="${prefix}base_link" link2="${prefix}link_1_s" reason="Adjacent"/>
